File: pulse-pcb/pulse-pcb.kicad_pcb (KiCad board)
At the start: 2 copper layers, 63.5 x 68.6 mm, 32 parts

Commit message: update
Connections:
- net Net-(A1-Pad15) renamed /STEP1
- net Net-(A1-Pad16) renamed /DIR1
- net Net-(A1-Pad2) renamed /+5V
