File: pulse-pcb/pulse-pcb.kicad_sch (KiCad schematic)
At the start: 9 parts

Commit message: update
Connections:
- net STEP1: now reaches A1.15 (STEP), N1.10 (D7)
- net DIR1: now reaches A1.16 (DIR), N1.11 (D8)
- net +5V: now reaches A1.2 (VDD), A2.2 (VDD), JPIR1.4 (Pin_4), N1.27 (+5V)
- net STEP2: now reaches A2.15 (STEP), N1.8 (D5)
- net DIR2: now reaches A2.16 (DIR), N1.9 (D6)
Changed lines of the file:
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@@
     (stroke (width 0) (type default) (color 0 0 0 0))
+  )
+  (label "DIR1" (at 92.71 115.57 0)
+    (effects (font (size 1.27 1.27)) (justify left bottom))
+  )
+  (label "+5V" (at 179.07 96.52 90)
+    (effects (font (size 1.27 1.27)) (justify left bottom))
+  )
+  (label "DIR2" (at 140.97 114.3 0)
+    (effects (font (size 1.27 1.27)) (justify left bottom))
+  )
+  (label "STEP1" (at 90.17 115.57 180)
+    (effects (font (size 1.27 1.27)) (justify right bottom))
   )
   (label "+12V" (at 176.53 69.85 180)
@@
     (effects (font (size 1.27 1.27)) (justify left bottom))
   )
+  (label "STEP2" (at 138.43 114.3 180)
+    (effects (font (size 1.27 1.27)) (justify right bottom))
+  )
   (symbol (lib_id "Connector:Screw_Terminal_01x04") (at 90.17 80.01 90) (unit 1)
